File: kicad/weather.sch (KiCad schematic (older format))
At the start: 14 parts, among them J1 Barrel_Jack, Q1 2N7000, U1 BME680

Commit message: 4060
Parts:
- added C4: 1n, Capacitor_SMD:C_1206_3216Metric_Pad1.33x1.80mm_HandSolder, symbol Device:C
- added C5: C, Capacitor_SMD:C_1206_3216Metric_Pad1.33x1.80mm_HandSolder, symbol Device:C
- added Q2: 2N7000, Package_TO_SOT_THT:TO-92_Inline, symbol Transistor_FET:2N7000
- added R5: 100k, Resistor_SMD:R_1206_3216Metric_Pad1.30x1.75mm_HandSolder, symbol Device:R_US
- added R6: 1M, Resistor_SMD:R_1206_3216Metric_Pad1.30x1.75mm_HandSolder, symbol Device:R_US
- added R7, R8, R9: R_US, Resistor_SMD:R_1206_3216Metric_Pad1.30x1.75mm_HandSolder, symbol Device:R_US
- added U2: CD4060BM96, Package_SO:SOIC-16_3.9x9.9mm_P1.27mm, symbol CD4060BM96:CD4060BM96
- U1: value BME680 -> BME280
Connections:
- net +3V3: now also R7.1, U2.16 (VDD)
- net GND: now also C5.2, Q2.1 (S), R9.2, U2.8 (GND)
- net at A1.1 (~RST), A1.4 (16): now also Q2.3 (D), R7.2
- new net: R5.2, U2.10 (CLK_0)
- new net: R6.2, U2.11 (CLK_1)
- new net: C5.1, R8.2, R9.1, U2.12 (RST)
- new net: Q2.2 (G), R8.1, U2.3 (Q14)
- new net: C4.1, U2.9 (CLK_0-1)
- new net: C4.2, R5.1, R6.1
- no-connect marks 14 -> 23
Other:
- note added: "ADAFRUIT 2652"
- note added: "AUTO-RESET TIMER\n(ONCE PER HOUR)"
- note added: "BME280"
- note added: "T\n= 2.3 R5 C4\n= 0.23 seconds"
- note removed: "ADAFRUIT 3660"
- note removed: "BME680"
- moved on the sheet: A1, D2, Q1, R2, R3, R4, U1

Commit message: revisionB
Parts:
- removed Q1, Q2: 2N7000, Package_TO_SOT_THT:TO-92_Inline, symbol Transistor_FET:2N7000
- added Q1, Q2: 2N7000, Package_TO_SOT_SMD:SOT-23_Handsoldering, symbol Device:Q_NMOS_GSD
Connections:
- net GND: now also Q1.2 (S), Q2.2 (S)
- net at A1.1 (~RST), A1.4 (16), R7.2: now also Q2.3 (D)
- net at A1.6 (12): now also Q1.1 (G)
- net at D2.1 (K): now also Q1.3 (D)
- net at R8.1, U2.3 (Q14): now also Q2.1 (G)
Changed lines of the file:
@@
 Sheet 1 1
 Title "MQTT Weather Station"
-Date "2021-04-07"
+Date "2021-04-12"
 Rev "B"
 Comp "University of Wisconsin-Madison"
@@
 $EndComp
 $Comp
-L Transistor_FET:2N7000 Q1
-U 1 1 5FCC5563
-P 9200 4000
-F 0 "Q1" H 9404 4046 50  0000 L CNN
-F 1 "2N7000" H 9404 3955 50  0000 L CNN
-F 2 "Package_TO_SOT_THT:TO-92_Inline" H 9400 3925 50  0001 L CIN
-F 3 "https://www.onsemi.com/pub/Collateral/NDS7002A-D.PDF" H 9200 4000 50  0001 L CNN
-	1    9200 4000
-	1    0    0    -1
-$EndComp
-$Comp
 L power:GND #PWR0105
 U 1 1 5FCC5CEE
@@
 Wire Wire Line
 	1150 1800 1150 2000
-Wire Wire Line
-	1150 2300 1500 2300
-Connection ~ 1500 2300
 NoConn ~ 2150 2300
 NoConn ~ 2150 2400
@@
 	5250 3200 6650 3200
 $Comp
-L Transistor_FET:2N7000 Q2
-U 1 1 6080DD81
-P 4200 2600
-F 0 "Q2" H 4404 2646 50  0000 L CNN
-F 1 "2N7000" H 4404 2555 50  0000 L CNN
-F 2 "Package_TO_SOT_THT:TO-92_Inline" H 4400 2525 50  0001 L CIN
-F 3 "https://www.onsemi.com/pub/Collateral/NDS7002A-D.PDF" H 4200 2600 50  0001 L CNN
-	1    4200 2600
-	1    0    0    -1
-$EndComp
-$Comp
 L Device:R_US R7
 U 1 1 6081A7E5
@@
 Wire Wire Line
 	4300 2400 5250 2400
-Connection ~ 4300 2400
 Connection ~ 5250 2400
 Wire Wire Line
@@
 Wire Wire Line
 	1850 2000 2150 2000
-Wire Wire Line
-	1500 2300 1850 2300
 $Comp
 L Device:R_US R6
@@
 $EndComp
 NoConn ~ 2150 2200
+$Comp
+L Device:Q_NMOS_GSD Q2
+U 1 1 607548BC
+P 4200 2600
+F 0 "Q2" H 4404 2646 50  0000 L CNN
+F 1 "2N7000" H 4404 2555 50  0000 L CNN
+F 2 "Package_TO_SOT_SMD:SOT-23_Handsoldering" H 4400 2700 50  0001 C CNN
+F 3 "~" H 4200 2600 50  0001 C CNN
+	1    4200 2600
+	1    0    0    -1
+$EndComp
+Connection ~ 4300 2400
+$Comp
+L Device:Q_NMOS_GSD Q1
+U 1 1 6075743A
+P 9200 4000
+F 0 "Q1" H 9404 4046 50  0000 L CNN
+F 1 "2N7000" H 9404 3955 50  0000 L CNN
+F 2 "Package_TO_SOT_SMD:SOT-23_Handsoldering" H 9400 4100 50  0001 C CNN
+F 3 "~" H 9200 4000 50  0001 C CNN
+	1    9200 4000
+	1    0    0    -1
+$EndComp
+Wire Wire Line
+	1150 2300 1500 2300
+Connection ~ 1500 2300
+Wire Wire Line
+	1500 2300 1850 2300
 $EndSCHEMATC

Commit message: after building one
Parts:
- R5: value 100k -> 470k
Other:
- note added: "AUTO-RESET TIMER\n(ONCE EVERY 2.5 HOUR)"
- note removed: "AUTO-RESET TIMER\n(ONCE PER HOUR)"
- note removed: "T\n= 2.3 R5 C4\n= 0.23 seconds"
Changed lines of the file:
@@
 Sheet 1 1
 Title "MQTT Weather Station"
-Date "2021-04-12"
+Date "2021-05-25"
 Rev "B"
 Comp "University of Wisconsin-Madison"
@@
 	1    0    0    -1
 $EndComp
-$Comp
-L Device:R_US R5
-U 1 1 606F2A08
-P 1150 2150
-F 0 "R5" H 1082 2104 50  0000 R CNN
-F 1 "100k" H 1082 2195 50  0000 R CNN
-F 2 "Resistor_SMD:R_1206_3216Metric_Pad1.30x1.75mm_HandSolder" V 1190 2140 50  0001 C CNN
-F 3 "~" H 1150 2150 50  0001 C CNN
-	1    1150 2150
-	-1   0    0    1
-$EndComp
 Wire Wire Line
 	2150 1900 1500 1900
@@
 NoConn ~ 3550 2500
 Text Notes 1050 1450 0    50   ~ 0
-AUTO-RESET TIMER\n(ONCE PER HOUR)
-Text Notes 1150 2750 0    50   ~ 0
-T\n= 2.3 R5 C4\n= 0.23 seconds
+AUTO-RESET TIMER\n(ONCE EVERY 2.5 HOUR)
 $Comp
 L CD4060BM96:CD4060BM96 U2
@@
 Wire Wire Line
 	1500 2300 1850 2300
+$Comp
+L Device:R_US R5
+U 1 1 606F2A08
+P 1150 2150
+F 0 "R5" H 1082 2104 50  0000 R CNN
+F 1 "470k" H 1082 2195 50  0000 R CNN
+F 2 "Resistor_SMD:R_1206_3216Metric_Pad1.30x1.75mm_HandSolder" V 1190 2140 50  0001 C CNN
+F 3 "~" H 1150 2150 50  0001 C CNN
+	1    1150 2150
+	-1   0    0    1
+$EndComp
 $EndSCHEMATC

Commit message: bom
Parts:
- C5: value C -> 1u
- R7, R8: value R_US -> 4.7k
- R9: value R_US -> 1M
Changed lines of the file:
@@
 P 4300 2250
 F 0 "R7" H 4368 2296 50  0000 L CNN
-F 1 "R_US" H 4368 2205 50  0000 L CNN
+F 1 "4.7k" H 4368 2205 50  0000 L CNN
 F 2 "Resistor_SMD:R_1206_3216Metric_Pad1.30x1.75mm_HandSolder" V 4340 2240 50  0001 C CNN
 F 3 "~" H 4300 2250 50  0001 C CNN
@@
 P 3200 3500
 F 0 "R8" V 3405 3500 50  0000 C CNN
-F 1 "R_US" V 3314 3500 50  0000 C CNN
+F 1 "4.7k" V 3314 3500 50  0000 C CNN
 F 2 "Resistor_SMD:R_1206_3216Metric_Pad1.30x1.75mm_HandSolder" V 3240 3490 50  0001 C CNN
 F 3 "~" H 3200 3500 50  0001 C CNN
@@
 P 2350 3650
 F 0 "C5" H 2465 3696 50  0000 L CNN
-F 1 "C" H 2465 3605 50  0000 L CNN
+F 1 "1u" H 2465 3605 50  0000 L CNN
 F 2 "Capacitor_SMD:C_1206_3216Metric_Pad1.33x1.80mm_HandSolder" H 2388 3500 50  0001 C CNN
 F 3 "~" H 2350 3650 50  0001 C CNN
@@
 Wire Wire Line
 	2350 3500 2650 3500
-$Comp
-L Device:R_US R9
-U 1 1 60872B34
-P 2650 3650
-F 0 "R9" H 2718 3696 50  0000 L CNN
-F 1 "R_US" H 2718 3605 50  0000 L CNN
-F 2 "Resistor_SMD:R_1206_3216Metric_Pad1.30x1.75mm_HandSolder" V 2690 3640 50  0001 C CNN
-F 3 "~" H 2650 3650 50  0001 C CNN
-	1    2650 3650
-	1    0    0    -1
-$EndComp
 Connection ~ 2650 3500
 Wire Wire Line
@@
 	-1   0    0    1
 $EndComp
+$Comp
+L Device:R_US R9
+U 1 1 60872B34
+P 2650 3650
+F 0 "R9" H 2718 3696 50  0000 L CNN
+F 1 "1M" H 2718 3605 50  0000 L CNN
+F 2 "Resistor_SMD:R_1206_3216Metric_Pad1.30x1.75mm_HandSolder" V 2690 3640 50  0001 C CNN
+F 3 "~" H 2650 3650 50  0001 C CNN
+	1    2650 3650
+	1    0    0    -1
+$EndComp
 $EndSCHEMATC

Commit message: c5
Parts:
- C4: value 1n -> 1u
Changed lines of the file:
@@
 Sheet 1 1
 Title "MQTT Weather Station"
-Date "2021-05-25"
-Rev "B"
+Date "2021-08-04"
+Rev "WIP"
 Comp "University of Wisconsin-Madison"
 Comment1 "Department of Chemistry"
@@
 P 1500 2150
 F 0 "C4" H 1615 2196 50  0000 L CNN
-F 1 "1n" H 1615 2105 50  0000 L CNN
+F 1 "1u" H 1615 2105 50  0000 L CNN
 F 2 "Capacitor_SMD:C_1206_3216Metric_Pad1.33x1.80mm_HandSolder" H 1538 2000 50  0001 C CNN
 F 3 "~" H 1500 2150 50  0001 C CNN
